Commit message: final

File: models/arm/standalone_arm.urdf.urdf (robot description, URDF)
Before this commit: robot my_robot, 13 links, 12 joints
Links:
- removed link base_footprint
- removed link base_link
- removed link camera_link
- removed link camera_link_optical
- removed link caster_wheel_link
- removed link left_wheel_link
- removed link right_wheel_link
Joints:
- removed joint base_camera_joint
- removed joint base_caster_wheel_joint
- removed joint base_joint
- removed joint base_left_wheel_joint
- removed joint base_right_wheel_joint
- removed joint camera_optical_joint
- removed joint mobile_base_arm_joint

File: models/urdf/common_properties.xacro (robot description, xacro)
@@ -1,18 +1,46 @@
 <?xml version="1.0"?>
 <robot xmlns:xacro="http://www.ros.org/wiki/xacro">
-    <material name="blue">
-        <color rgba="0 0 0.5 1" />
-    </material>
     <material name="grey">
         <color rgba="0.5 0.5 0.5 1" />
     </material>
+    <!-- Red Material -->
+    <material name="red">
+        <color rgba="1 0 0 1" />
+    </material>
+    <!-- Green Material -->
+    <material name="green">
+        <color rgba="0 1 0 1" />
+    </material>
+    <!-- Blue Material -->
+    <material name="blue">
+        <color rgba="0 0 1 1" />
+    </material>
+    <!-- Yellow Material -->
+    <material name="yellow">
+        <color rgba="1 1 0 1" />
+    </material>
+    <!-- Purple Material -->
+    <material name="purple">
+        <color rgba="0.5 0 0.5 1" />
+    </material>
+    <!-- Orange Material -->
+    <material name="orange">
+        <color rgba="1 0.5 0 1" />
+    </material>
+    <!-- Cyan Material -->
+    <material name="cyan">
+        <color rgba="0 1 1 1" />
+    </material>
+    <!-- Magenta Material -->
+    <material name="magenta">
+        <color rgba="1 0 1 1" />
+    </material>
+    <!-- White Material -->
+    <material name="white">
+        <color rgba="1 1 1 1" />
+    </material>
+    <!-- Black Material -->
     <material name="black">
-        <color rgba="0.0 0.0 0.0 1" />
-    </material>
-    <material name="orange">
-        <color rgba="1.0 0.5 0 1" />
-    </material>
-    <material name="yellow">
-        <color rgba="1.0 1.0 0 1" />
+        <color rgba="0 0 0 1" />
     </material>
     <xacro:macro name="box_inertia" params="m l w h xyz rpy">
